File: PCB/Prototype Board.sch (EAGLE design)
At the start: 78 parts, among them Q1 S8050, Q10 20V/0.2A/8MHz/1.2Ω/1Vth, Q2 20V/0.2A/8MHz/1.2Ω/1Vth, Q3 20V/4.2A/52mΩ/1.4W, Q4 S8050, Q5 20V/0.2A/8MHz/1.2Ω/1Vth, Q6 20V/0.2A/8MHz/1.2Ω/1Vth, Q7 20V/0.2A/8MHz/1.2Ω/1Vth, Q8 20V/0.2A/8MHz/1.2Ω/1Vth, U1 9DoF IMU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

Commit message: Finalized PCB
Parts:
- removed U1: 9DoF IMU, SparkFun-Sensors:ICM-20948
- added U$12: ICM20948, customlib:ICM20948
Connections:
- net 1.8V: now also U$12.VDD, U$12.VDDIO; no longer U1.VDD, U1.VDDIO
- net FSYNC/IO36: now also U$12.FSYNC; no longer U1.FSYNC
- net GND: now also U$12.GND, U3.GND; no longer U1.GND
- net GPIO12/SDO: now also U$12.AD0/SD0; no longer U1.AD0/SDO
- net GPIO13/SDI: now also U$12.SDA/SDI; no longer U1.SDA/SDI
- net GPIO14/SCLK: now also U$12.SCL/SCLK; no longer U1.SCL/SCLK
- net GPIO15/CS: now also U$12.CS; no longer U1.!CS
- net INT/IO39: now also U$12.INT; no longer U1.INT
- net N$13: now also U$12.REGOUT; no longer U1.REGOUT
Changed lines of the file:
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@@
 <part name="SUPPLY3" library="SparkFun-PowerSymbols" deviceset="3.3V" device=""/>
 <part name="GND6" library="SparkFun-PowerSymbols" deviceset="GND" device=""/>
-<part name="U1" library="SparkFun-Sensors" deviceset="ICM-20948" device="" value="9DoF IMU"/>
 <part name="SUPPLY8" library="SparkFun-PowerSymbols" deviceset="VIN" device=""/>
 <part name="GND12" library="SparkFun-PowerSymbols" deviceset="GND" device=""/>
@@
 <part name="R7" library="JLC PCB Basic Parts_loc" deviceset="R_" device="_0603" package3d_urn="urn:adsk.eagle:package:23555/3" technology="4.7K"/>
 <part name="U$8" library="customlib" deviceset="SM02B_PASS_TB_LF" device=""/>
-<part name="U$6" library="customlib" deviceset="19-217/GHC-YR1S2/3T" device=""/>
 <part name="GND7" library="SparkFun-PowerSymbols" deviceset="GND" device=""/>
-<part name="U$9" library="customlib" deviceset="19-217/GHC-YR1S2/3T" device=""/>
 <part name="U5" library="DWM1000" deviceset="DWM1000" device=""/>
 <part name="GND8" library="SparkFun-PowerSymbols" deviceset="GND" device=""/>
@@
 <part name="SUPPLY30" library="SparkFun-PowerSymbols" deviceset="3.3V" device=""/>
 <part name="GND5" library="SparkFun-PowerSymbols" deviceset="GND" device=""/>
+<part name="U$6" library="customlib" deviceset="19-217/GHC-YR1S2/3T" device=""/>
+<part name="U$9" library="customlib" deviceset="19-217/GHC-YR1S2/3T" device=""/>
+<part name="U$12" library="customlib" deviceset="ICM20948" device=""/>
 </parts>
 <sheets>
@@
 <attribute name="VALUE" x="289.56" y="144.526" size="1.778" layer="96" align="top-center"/>
 </instance>
-<instance part="U1" gate="G$1" x="147.32" y="116.84" smashed="yes">
-<attribute name="NAME" x="134.62" y="127.254" size="1.778" layer="95" font="vector"/>
-<attribute name="VALUE" x="134.62" y="108.966" size="1.778" layer="96" font="vector" align="top-left"/>
-</instance>
 <instance part="SUPPLY8" gate="G$1" x="210.82" y="279.4" smashed="yes"/>
 <instance part="GND12" gate="1" x="210.82" y="251.46" smashed="yes">
@@
 <attribute name="VALUE" x="109.22" y="279.4" size="1.778" layer="96" font="vector"/>
 </instance>
-<instance part="GND58" gate="1" x="200.66" y="248.92" smashed="yes">
-<attribute name="VALUE" x="200.66" y="248.666" size="1.778" layer="96" align="top-center"/>
+<instance part="GND58" gate="1" x="200.66" y="243.84" smashed="yes">
+<attribute name="VALUE" x="200.66" y="243.586" size="1.778" layer="96" align="top-center"/>
 </instance>
 <instance part="GND10" gate="1" x="-12.7" y="139.7" smashed="yes">
@@
 </instance>
 <instance part="U$8" gate="G$1" x="60.96" y="279.4" smashed="yes"/>
-<instance part="U$6" gate="G$1" x="0" y="266.7" smashed="yes" rot="R90"/>
 <instance part="GND7" gate="1" x="220.98" y="259.08" smashed="yes">
 <attribute name="VALUE" x="220.98" y="258.826" size="1.778" layer="96" align="top-center"/>
 </instance>
-<instance part="U$9" gate="G$1" x="200.66" y="259.08" smashed="yes" rot="R270"/>
 <instance part="U5" gate="G$1" x="147.32" y="139.7" smashed="yes"/>
 <instance part="GND8" gate="1" x="172.72" y="144.78" smashed="yes">
@@
 <attribute name="VALUE" x="254" y="180.594" size="1.778" layer="96" rot="R180" align="top-center"/>
 </instance>
+<instance part="U$6" gate="G$1" x="0" y="266.7" smashed="yes" rot="R90"/>
+<instance part="U$9" gate="G$1" x="200.66" y="256.54" smashed="yes" rot="R270"/>
+<instance part="U$12" gate="G$1" x="147.32" y="119.38" smashed="yes"/>
 </instances>
 <busses>
@@
 <wire x1="66.04" y1="158.75" x2="81.28" y2="158.75" width="0.1524" layer="91"/>
 <wire x1="81.28" y1="158.75" x2="81.28" y2="160.02" width="0.1524" layer="91"/>
+<pinref part="U3" gate="G$1" pin="GND"/>
+<wire x1="43.18" y1="138.43" x2="43.18" y2="158.75" width="0.1524" layer="91"/>
+<wire x1="43.18" y1="158.75" x2="66.04" y2="158.75" width="0.1524" layer="91"/>
+<junction x="66.04" y="158.75"/>
 </segment>
 <segment>
@@
 </segment>
 <segment>
-<pinref part="U1" gate="G$1" pin="GND"/>
 <wire x1="132.08" y1="111.76" x2="127" y2="111.76" width="0.1524" layer="91"/>
 <pinref part="GND17" gate="1" pin="GND"/>
 <wire x1="127" y1="111.76" x2="127" y2="104.14" width="0.1524" layer="91"/>
 <wire x1="127" y1="104.14" x2="125.73" y2="104.14" width="0.1524" layer="91"/>
+<pinref part="U$12" gate="G$1" pin="GND"/>
 </segment>
 <segment>
@@
 <wire x1="220.98" y1="264.16" x2="220.98" y2="261.62" width="0.1524" layer="91"/>
 <pinref part="GND7" gate="1" pin="GND"/>
-</segment>
-<segment>
-<pinref part="U$9" gate="G$1" pin="2"/>
-<pinref part="GND58" gate="1" pin="GND"/>
 </segment>
 <segment>
@@
 <pinref part="GND5" gate="1" pin="GND"/>
 <pinref part="U$11" gate="G$1" pin="GND"/>
+</segment>
+<segment>
+<pinref part="U$9" gate="G$1" pin="2"/>
+<pinref part="GND58" gate="1" pin="GND"/>
+<wire x1="200.66" y1="246.38" x2="200.66" y2="248.92" width="0.1524" layer="91"/>
 </segment>
 </net>
@@
 </segment>
 <segment>
-<pinref part="U1" gate="G$1" pin="VDD"/>
 <wire x1="132.08" y1="124.46" x2="116.84" y2="124.46" width="0.1524" layer="91"/>
 <wire x1="116.84" y1="124.46" x2="109.22" y2="124.46" width="0.1524" layer="91"/>
 <wire x1="109.22" y1="124.46" x2="109.22" y2="114.3" width="0.1524" layer="91"/>
-<pinref part="U1" gate="G$1" pin="VDDIO"/>
 <wire x1="132.08" y1="121.92" x2="116.84" y2="121.92" width="0.1524" layer="91"/>
 <wire x1="116.84" y1="121.92" x2="116.84" y2="124.46" width="0.1524" layer="91"/>
@@
 <pinref part="C6" gate="G$1" pin="1"/>
 <pinref part="C8" gate="G$1" pin="1"/>
+<pinref part="U$12" gate="G$1" pin="VDD"/>
+<pinref part="U$12" gate="G$1" pin="VDDIO"/>
 </segment>
 <segment>
@@
 <net name="N$13" class="0">
 <segment>
-<pinref part="U1" gate="G$1" pin="REGOUT"/>
 <wire x1="132.08" y1="114.3" x2="116.84" y2="114.3" width="0.1524" layer="91"/>
 <pinref part="C9" gate="G$1" pin="1"/>
+<pinref part="U$12" gate="G$1" pin="REGOUT"/>
 </segment>
 </net>
 <net name="GPIO15/CS" class="0">
 <segment>
-<pinref part="U1" gate="G$1" pin="!CS"/>
 <wire x1="162.56" y1="119.38" x2="170.18" y2="119.38" width="0.1524" layer="91"/>
 <label x="170.18" y="119.38" size="1.778" layer="95"/>
+<pinref part="U$12" gate="G$1" pin="CS"/>
 </segment>
 <segment>
@@
 <net name="GPIO14/SCLK" class="0">
 <segment>
-<pinref part="U1" gate="G$1" pin="SCL/SCLK"/>
 <wire x1="162.56" y1="116.84" x2="170.18" y2="116.84" width="0.1524" layer="91"/>
 <label x="170.18" y="116.84" size="1.778" layer="95"/>
+<pinref part="U$12" gate="G$1" pin="SCL/SCLK"/>
 </segment>
 <segment>
@@
 <net name="GPIO13/SDI" class="0">
 <segment>
-<pinref part="U1" gate="G$1" pin="SDA/SDI"/>
 <wire x1="162.56" y1="114.3" x2="170.18" y2="114.3" width="0.1524" layer="91"/>
 <label x="170.18" y="114.3" size="1.778" layer="95"/>
+<pinref part="U$12" gate="G$1" pin="SDA/SDI"/>
 </segment>
 <segment>
@@
 <net name="GPIO12/SDO" class="0">
 <segment>
-<pinref part="U1" gate="G$1" pin="AD0/SDO"/>
 <wire x1="162.56" y1="111.76" x2="170.18" y2="111.76" width="0.1524" layer="91"/>
 <label x="170.18" y="111.76" size="1.778" layer="95"/>
+<pinref part="U$12" gate="G$1" pin="AD0/SD0"/>
 </segment>
 <segment>
@@
 <net name="INT/IO39" class="0">
 <segment>
-<pinref part="U1" gate="G$1" pin="INT"/>
 <wire x1="132.08" y1="119.38" x2="124.46" y2="119.38" width="0.1524" layer="91"/>
 <label x="121.92" y="119.38" size="1.778" layer="95"/>
+<pinref part="U$12" gate="G$1" pin="INT"/>
 </segment>
 <segment>
@@
 <net name="FSYNC/IO36" class="0">
 <segment>
-<pinref part="U1" gate="G$1" pin="FSYNC"/>
 <wire x1="132.08" y1="116.84" x2="124.46" y2="116.84" width="0.1524" layer="91"/>
 <label x="119.38" y="116.84" size="1.778" layer="95"/>
+<pinref part="U$12" gate="G$1" pin="FSYNC"/>
 </segment>
 <segment>
@@
 </segment>
 </net>
-<net name="N$4" class="0">
-<segment>
-<pinref part="U$9" gate="G$1" pin="1"/>
-<pinref part="R8" gate="R1" pin="1"/>
-</segment>
-</net>
 <net name="N$10" class="0">
 <segment>
@@
 </segment>
 </net>
+<net name="N$4" class="0">
+<segment>
+<pinref part="U$9" gate="G$1" pin="1"/>
+<pinref part="R8" gate="R1" pin="1"/>
+<wire x1="200.66" y1="264.16" x2="200.66" y2="266.7" width="0.1524" layer="91"/>
+</segment>
+</net>
